File: circuit2.sch (EAGLE design)
At the start: 16 parts, among them IC1 ATMEGA328-20P, IC2 786TV

Commit message: Add files via upload
Parts:
- removed C3: (no value), capacitor-wima:C2.5/2
- removed C4: 10u, capacitor-wima:C2.5/2
- removed IC2: 786TV, linear:786TV
- G1: value AB9V -> CR2430H; device battery:AB9V -> battery:CR2430H
Connections:
- removed net N$2: C4.1, IC2.GND
- removed net N$3: C3.1, G1.-
- new net N$16: IC1.(PCI2/SS/OC1B)PB2
- net GND: now also G1.-, SG1.2; no longer C3.2, C4.2
- net N$1: now also IC1.(PCI23/AIN1)PD7, SG1.1; no longer G1.+, IC2.VI
- net VCC: now also G1.+; no longer IC2.VO
Changed lines of the file:
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@@
 </variantdefs>
 <classes>
-<class number="0" name="default" width="0" drill="0">
+<class number="0" name="default" width="0.5" drill="0">
+</class>
+<class number="1" name="New Class" width="1.5" drill="0">
 </class>
 </classes>
@@
 <part name="IC1" library="atmega328" deviceset="ATMEGA328*P" device="" technology="-20"/>
 <part name="Q1" library="special" library_urn="urn:adsk.eagle:library:367" deviceset="XTAL/S" device="" package3d_urn="urn:adsk.eagle:package:26647/2"/>
-<part name="IC2" library="linear" library_urn="urn:adsk.eagle:library:262" deviceset="78*" device="TV" package3d_urn="urn:adsk.eagle:package:16417/2" technology="6"/>
 <part name="C1" library="capacitor-wima" library_urn="urn:adsk.eagle:library:116" deviceset="C" device="2.5/2" package3d_urn="urn:adsk.eagle:package:5415/1"/>
 <part name="C2" library="capacitor-wima" library_urn="urn:adsk.eagle:library:116" deviceset="C" device="2.5/2" package3d_urn="urn:adsk.eagle:package:5415/1"/>
-<part name="C3" library="capacitor-wima" library_urn="urn:adsk.eagle:library:116" deviceset="C" device="2.5/2" package3d_urn="urn:adsk.eagle:package:5415/1"/>
-<part name="C4" library="capacitor-wima" library_urn="urn:adsk.eagle:library:116" deviceset="C" device="2.5/2" package3d_urn="urn:adsk.eagle:package:5415/1" value="10u"/>
-<part name="G1" library="battery" library_urn="urn:adsk.eagle:library:109" deviceset="AB9V" device="" package3d_urn="urn:adsk.eagle:package:4600/1"/>
-<part name="P+1" library="supply1" library_urn="urn:adsk.eagle:library:371" deviceset="VCC" device=""/>
-<part name="GND1" library="supply1" library_urn="urn:adsk.eagle:library:371" deviceset="GND" device=""/>
 <part name="TR1" library="discrete" library_urn="urn:adsk.eagle:library:211" deviceset="THERMISTOR_" device="R-5" package3d_urn="urn:adsk.eagle:package:12931/1" value="10k"/>
 <part name="TR2" library="discrete" library_urn="urn:adsk.eagle:library:211" deviceset="THERMISTOR_" device="R-5" package3d_urn="urn:adsk.eagle:package:12931/1"/>
@@
 <part name="GND9" library="supply1" library_urn="urn:adsk.eagle:library:371" deviceset="GND" device=""/>
 <part name="SG1" library="buzzer" library_urn="urn:adsk.eagle:library:113" deviceset="B/C11L" device="" package3d_urn="urn:adsk.eagle:package:5280/1"/>
+<part name="GND10" library="supply1" library_urn="urn:adsk.eagle:library:371" deviceset="GND" device=""/>
+<part name="G1" library="battery" library_urn="urn:adsk.eagle:library:109" deviceset="CR2430H" device="" package3d_urn="urn:adsk.eagle:package:4583/1"/>
+<part name="P+1" library="supply1" library_urn="urn:adsk.eagle:library:371" deviceset="VCC" device=""/>
+<part name="GND1" library="supply1" library_urn="urn:adsk.eagle:library:371" deviceset="GND" device=""/>
 </parts>
 <sheets>
@@
 <attribute name="VALUE" x="-21.59" y="34.29" size="1.778" layer="96" rot="R90"/>
 </instance>
-<instance part="IC2" gate="A1" x="68.58" y="-21.59" smashed="yes">
-<attribute name="NAME" x="60.96" y="-15.875" size="1.778" layer="95"/>
-<attribute name="VALUE" x="60.96" y="-18.415" size="1.778" layer="96"/>
-</instance>
 <instance part="C1" gate="G$1" x="-31.75" y="25.4" smashed="yes" rot="R90">
 <attribute name="NAME" x="-32.131" y="26.924" size="1.778" layer="95" rot="R90"/>
@@
 <attribute name="VALUE" x="-27.051" y="56.134" size="1.778" layer="96" rot="R90"/>
 </instance>
-<instance part="C3" gate="G$1" x="31.75" y="-34.29" smashed="yes">
-<attribute name="NAME" x="33.274" y="-33.909" size="1.778" layer="95"/>
-<attribute name="VALUE" x="33.274" y="-38.989" size="1.778" layer="96"/>
-</instance>
-<instance part="C4" gate="G$1" x="68.58" y="-34.29" smashed="yes">
-<attribute name="NAME" x="70.104" y="-33.909" size="1.778" layer="95"/>
-<attribute name="VALUE" x="70.104" y="-38.989" size="1.778" layer="96"/>
-</instance>
-<instance part="G1" gate="G$1" x="44.45" y="-21.59" smashed="yes">
-<attribute name="NAME" x="38.735" y="-18.415" size="1.778" layer="95"/>
-<attribute name="VALUE" x="38.735" y="-26.67" size="1.778" layer="96"/>
-</instance>
-<instance part="P+1" gate="VCC" x="80.01" y="-15.24" smashed="yes">
-<attribute name="VALUE" x="77.47" y="-17.78" size="1.778" layer="96" rot="R90"/>
-</instance>
-<instance part="GND1" gate="1" x="44.45" y="-44.45" smashed="yes">
-<attribute name="VALUE" x="41.91" y="-46.99" size="1.778" layer="96"/>
-</instance>
 <instance part="TR1" gate="G$1" x="-19.05" y="63.5" smashed="yes">
 <attribute name="NAME" x="-21.59" y="67.31" size="1.778" layer="95"/>
@@
 <attribute name="NAME" x="96.52" y="34.29" size="1.778" layer="95"/>
 <attribute name="VALUE" x="105.41" y="27.94" size="1.778" layer="96"/>
+</instance>
+<instance part="GND10" gate="1" x="104.14" y="20.32" smashed="yes">
+<attribute name="VALUE" x="101.6" y="17.78" size="1.778" layer="96"/>
+</instance>
+<instance part="G1" gate="1" x="48.26" y="-25.4" smashed="yes">
+<attribute name="NAME" x="45.72" y="-22.225" size="1.778" layer="95"/>
+<attribute name="VALUE" x="45.72" y="-30.48" size="1.778" layer="96"/>
+</instance>
+<instance part="P+1" gate="VCC" x="58.42" y="-20.32" smashed="yes">
+<attribute name="VALUE" x="55.88" y="-22.86" size="1.778" layer="96" rot="R90"/>
+</instance>
+<instance part="GND1" gate="1" x="40.64" y="-30.48" smashed="yes">
+<attribute name="VALUE" x="38.1" y="-33.02" size="1.778" layer="96"/>
 </instance>
 </instances>
@@
 </busses>
 <nets>
-<net name="N$1" class="0">
-<segment>
-<pinref part="G1" gate="G$1" pin="+"/>
-<pinref part="IC2" gate="A1" pin="VI"/>
-<wire x1="57.15" y1="-21.59" x2="58.42" y2="-21.59" width="0.1524" layer="91"/>
-</segment>
-</net>
-<net name="VCC" class="0">
-<segment>
-<pinref part="P+1" gate="VCC" pin="VCC"/>
-<pinref part="IC2" gate="A1" pin="VO"/>
-<wire x1="80.01" y1="-17.78" x2="80.01" y2="-21.59" width="0.1524" layer="91"/>
-<wire x1="80.01" y1="-21.59" x2="78.74" y2="-21.59" width="0.1524" layer="91"/>
-</segment>
+<net name="VCC" class="1">
 <segment>
 <pinref part="P+2" gate="VCC" pin="VCC"/>
@@
 <wire x1="127" y1="22.86" x2="127" y2="25.4" width="0.1524" layer="91"/>
 </segment>
-</net>
-<net name="GND" class="0">
-<segment>
-<wire x1="31.75" y1="-40.64" x2="44.45" y2="-40.64" width="0.1524" layer="91"/>
-<wire x1="44.45" y1="-40.64" x2="68.58" y2="-40.64" width="0.1524" layer="91"/>
-<pinref part="GND1" gate="1" pin="GND"/>
-<wire x1="44.45" y1="-41.91" x2="44.45" y2="-40.64" width="0.1524" layer="91"/>
-<junction x="44.45" y="-40.64"/>
-<wire x1="68.58" y1="-40.64" x2="68.58" y2="-39.37" width="0.1524" layer="91"/>
-<pinref part="C4" gate="G$1" pin="2"/>
-<wire x1="31.75" y1="-39.37" x2="31.75" y2="-40.64" width="0.1524" layer="91"/>
-<pinref part="C3" gate="G$1" pin="2"/>
-</segment>
+<segment>
+<pinref part="G1" gate="1" pin="+"/>
+<pinref part="P+1" gate="VCC" pin="VCC"/>
+<wire x1="53.34" y1="-25.4" x2="58.42" y2="-25.4" width="0.1524" layer="91"/>
+<wire x1="58.42" y1="-25.4" x2="58.42" y2="-22.86" width="0.1524" layer="91"/>
+</segment>
+</net>
+<net name="GND" class="1">
 <segment>
 <pinref part="C2" gate="G$1" pin="1"/>
@@
 <wire x1="147.32" y1="27.94" x2="147.32" y2="22.86" width="0.1524" layer="91"/>
 </segment>
-</net>
-<net name="N$2" class="0">
-<segment>
-<pinref part="IC2" gate="A1" pin="GND"/>
-<wire x1="68.58" y1="-31.75" x2="68.58" y2="-29.21" width="0.1524" layer="91"/>
-<pinref part="C4" gate="G$1" pin="1"/>
-</segment>
-</net>
-<net name="N$3" class="0">
-<segment>
-<pinref part="G1" gate="G$1" pin="-"/>
-<wire x1="31.75" y1="-21.59" x2="31.75" y2="-31.75" width="0.1524" layer="91"/>
-<pinref part="C3" gate="G$1" pin="1"/>
+<segment>
+<pinref part="GND1" gate="1" pin="GND"/>
+<pinref part="G1" gate="1" pin="-"/>
+<wire x1="40.64" y1="-27.94" x2="43.18" y2="-27.94" width="0.1524" layer="91"/>
+<wire x1="43.18" y1="-27.94" x2="43.18" y2="-25.4" width="0.1524" layer="91"/>
+</segment>
+<segment>
+<pinref part="SG1" gate="G$1" pin="2"/>
+<pinref part="GND10" gate="1" pin="GND"/>
+<wire x1="104.14" y1="25.4" x2="104.14" y2="22.86" width="0.1524" layer="91"/>
 </segment>
 </net>
@@
 </segment>
 </net>
+<net name="N$16" class="0">
+<segment>
+<pinref part="IC1" gate="G$1" pin="(PCI2/SS/OC1B)PB2"/>
+<wire x1="50.8" y1="10.16" x2="96.52" y2="10.16" width="0.1524" layer="91"/>
+</segment>
+</net>
+<net name="N$1" class="0">
+<segment>
+<pinref part="IC1" gate="G$1" pin="(PCI23/AIN1)PD7"/>
+<pinref part="SG1" gate="G$1" pin="1"/>
+<wire x1="50.8" y1="20.32" x2="96.52" y2="20.32" width="0.1524" layer="91"/>
+<wire x1="96.52" y1="20.32" x2="96.52" y2="25.4" width="0.1524" layer="91"/>
+</segment>
+</net>

Commit message: Adição dos modelos 3D dos principais componentes
Parts:
- removed S2: TL32PO, switch:TL32PO
- added S1: DT6, switch-misc:DT6
- S3: value DTS-6 -> (none); device switch-tact:DTS-6 -> switch:320-916
- SG1: value B/C11L -> F/CM12P; device buzzer:B/C11L -> buzzer:F/CM12P
Connections:
- net GND: now also S3.P; no longer S2.P
- net N$17: now also S1.P@1; no longer S3.2
- net N$19: now also S1.S@1; no longer S3.4
- net N$4: now also S3.O; no longer S2.O
- net VCC: now also S1.P; no longer S3.1
Changed lines of the file:
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@@
 </classes>
 <parts>
-<part name="IC1" library="atmega328" deviceset="ATMEGA328*P" device="" technology="-20"/>
+<part name="IC1" library="atmega328" deviceset="ATMEGA328*P" device="" override_package3d_urn="urn:adsk.eagle:package:34532548/2" override_package_urn="urn:adsk.eagle:footprint:34532549/1" technology="-20"/>
 <part name="Q1" library="special" library_urn="urn:adsk.eagle:library:367" deviceset="XTAL/S" device="" package3d_urn="urn:adsk.eagle:package:26647/2"/>
 <part name="C1" library="capacitor-wima" library_urn="urn:adsk.eagle:library:116" deviceset="C" device="2.5/2" package3d_urn="urn:adsk.eagle:package:5415/1"/>
@@
 <part name="GND5" library="supply1" library_urn="urn:adsk.eagle:library:371" deviceset="GND" device=""/>
 <part name="GND6" library="supply1" library_urn="urn:adsk.eagle:library:371" deviceset="GND" device=""/>
-<part name="DIS1" library="display-lcd" library_urn="urn:adsk.eagle:library:214" deviceset="TUXGR_16X2_R2" device="" package3d_urn="urn:adsk.eagle:package:13139/1"/>
+<part name="DIS1" library="display-lcd" library_urn="urn:adsk.eagle:library:214" deviceset="TUXGR_16X2_R2" device="" package3d_urn="urn:adsk.eagle:package:13139/1" override_package3d_urn="urn:adsk.eagle:package:34532442/2" override_package_urn="urn:adsk.eagle:footprint:13120/1"/>
 <part name="GND7" library="supply1" library_urn="urn:adsk.eagle:library:371" deviceset="GND" device=""/>
 <part name="GND8" library="supply1" library_urn="urn:adsk.eagle:library:371" deviceset="GND" device=""/>
 <part name="P+5" library="supply1" library_urn="urn:adsk.eagle:library:371" deviceset="VCC" device=""/>
 <part name="P+6" library="supply1" library_urn="urn:adsk.eagle:library:371" deviceset="VCC" device=""/>
-<part name="S2" library="switch" library_urn="urn:adsk.eagle:library:380" deviceset="TL32PO" device="" package3d_urn="urn:adsk.eagle:package:27745/1"/>
-<part name="S3" library="switch-tact" deviceset="DTS-6" device=""/>
 <part name="P+7" library="supply1" library_urn="urn:adsk.eagle:library:371" deviceset="VCC" device=""/>
 <part name="GND9" library="supply1" library_urn="urn:adsk.eagle:library:371" deviceset="GND" device=""/>
-<part name="SG1" library="buzzer" library_urn="urn:adsk.eagle:library:113" deviceset="B/C11L" device="" package3d_urn="urn:adsk.eagle:package:5280/1"/>
 <part name="GND10" library="supply1" library_urn="urn:adsk.eagle:library:371" deviceset="GND" device=""/>
 <part name="G1" library="battery" library_urn="urn:adsk.eagle:library:109" deviceset="CR2430H" device="" package3d_urn="urn:adsk.eagle:package:4583/1"/>
 <part name="P+1" library="supply1" library_urn="urn:adsk.eagle:library:371" deviceset="VCC" device=""/>
 <part name="GND1" library="supply1" library_urn="urn:adsk.eagle:library:371" deviceset="GND" device=""/>
+<part name="S1" library="switch-misc" library_urn="urn:adsk.eagle:library:376" deviceset="DT" device="6" package3d_urn="urn:adsk.eagle:package:27430/1" override_package3d_urn="urn:adsk.eagle:package:34532255/2" override_package_urn="urn:adsk.eagle:footprint:27398/1"/>
+<part name="S3" library="switch" library_urn="urn:adsk.eagle:library:380" deviceset="320-916" device="" package3d_urn="urn:adsk.eagle:package:27678/1" override_package3d_urn="urn:adsk.eagle:package:34532324/2" override_package_urn="urn:adsk.eagle:footprint:27534/1"/>
+<part name="SG1" library="buzzer" library_urn="urn:adsk.eagle:library:113" deviceset="F/CM12P" device="" package3d_urn="urn:adsk.eagle:package:5265/1" override_package3d_urn="urn:adsk.eagle:package:34532438/2" override_package_urn="urn:adsk.eagle:footprint:5223/1"/>
 </parts>
 <sheets>
@@
 <attribute name="VALUE" x="71.12" y="60.96" size="1.778" layer="96" rot="R90"/>
 </instance>
-<instance part="S2" gate="BEF1" x="-27.94" y="71.12" smashed="yes" rot="R270">
-<attribute name="NAME" x="-30.48" y="66.04" size="1.778" layer="95"/>
-<attribute name="VALUE" x="-30.48" y="63.5" size="1.778" layer="96"/>
-</instance>
-<instance part="S3" gate="G$1" x="132.08" y="35.56" smashed="yes">
-<attribute name="NAME" x="125.73" y="33.02" size="1.778" layer="95" rot="R90"/>
-<attribute name="VALUE" x="128.27" y="38.735" size="1.778" layer="96" rot="R90"/>
-</instance>
 <instance part="P+7" gate="VCC" x="127" y="27.94" smashed="yes">
 <attribute name="VALUE" x="124.46" y="25.4" size="1.778" layer="96" rot="R90"/>
@@
 <instance part="GND9" gate="1" x="147.32" y="20.32" smashed="yes">
 <attribute name="VALUE" x="144.78" y="17.78" size="1.778" layer="96"/>
+</instance>
+<instance part="GND10" gate="1" x="104.14" y="20.32" smashed="yes">
+<attribute name="VALUE" x="101.6" y="17.78" size="1.778" layer="96"/>
+</instance>
+<instance part="G1" gate="1" x="48.26" y="-25.4" smashed="yes">
+<attribute name="NAME" x="45.72" y="-22.225" size="1.778" layer="95"/>
+<attribute name="VALUE" x="45.72" y="-30.48" size="1.778" layer="96"/>
+</instance>
+<instance part="P+1" gate="VCC" x="58.42" y="-20.32" smashed="yes">
+<attribute name="VALUE" x="55.88" y="-22.86" size="1.778" layer="96" rot="R90"/>
+</instance>
+<instance part="GND1" gate="1" x="40.64" y="-30.48" smashed="yes">
+<attribute name="VALUE" x="38.1" y="-33.02" size="1.778" layer="96"/>
+</instance>
+<instance part="S1" gate="1" x="132.08" y="35.56" smashed="yes">
+<attribute name="NAME" x="125.095" y="33.655" size="1.778" layer="95" rot="R90"/>
+<attribute name="VALUE" x="127.635" y="38.1" size="1.778" layer="96" rot="R90"/>
+</instance>
+<instance part="S3" gate="1" x="-27.94" y="73.66" smashed="yes" rot="R270">
+<attribute name="NAME" x="-29.845" y="80.01" size="1.778" layer="95"/>
+<attribute name="VALUE" x="-25.4" y="77.47" size="1.778" layer="96"/>
 </instance>
 <instance part="SG1" gate="G$1" x="99.06" y="27.94" smashed="yes">
 <attribute name="NAME" x="96.52" y="34.29" size="1.778" layer="95"/>
 <attribute name="VALUE" x="105.41" y="27.94" size="1.778" layer="96"/>
-</instance>
-<instance part="GND10" gate="1" x="104.14" y="20.32" smashed="yes">
-<attribute name="VALUE" x="101.6" y="17.78" size="1.778" layer="96"/>
-</instance>
-<instance part="G1" gate="1" x="48.26" y="-25.4" smashed="yes">
-<attribute name="NAME" x="45.72" y="-22.225" size="1.778" layer="95"/>
-<attribute name="VALUE" x="45.72" y="-30.48" size="1.778" layer="96"/>
-</instance>
-<instance part="P+1" gate="VCC" x="58.42" y="-20.32" smashed="yes">
-<attribute name="VALUE" x="55.88" y="-22.86" size="1.778" layer="96" rot="R90"/>
-</instance>
-<instance part="GND1" gate="1" x="40.64" y="-30.48" smashed="yes">
-<attribute name="VALUE" x="38.1" y="-33.02" size="1.778" layer="96"/>
 </instance>
 </instances>
@@
 </segment>
 <segment>
-<pinref part="S3" gate="G$1" pin="1"/>
 <wire x1="132.08" y1="30.48" x2="132.08" y2="22.86" width="0.1524" layer="91"/>
 <wire x1="132.08" y1="22.86" x2="127" y2="22.86" width="0.1524" layer="91"/>
 <pinref part="P+7" gate="VCC" pin="VCC"/>
 <wire x1="127" y1="22.86" x2="127" y2="25.4" width="0.1524" layer="91"/>
+<pinref part="S1" gate="1" pin="P"/>
 </segment>
 <segment>
@@
 <segment>
 <pinref part="GND2" gate="1" pin="GND"/>
-<pinref part="S2" gate="BEF1" pin="P"/>
 <wire x1="-35.56" y1="68.58" x2="-35.56" y2="71.12" width="0.1524" layer="91"/>
 <wire x1="-35.56" y1="71.12" x2="-33.02" y2="71.12" width="0.1524" layer="91"/>
+<pinref part="S3" gate="1" pin="P"/>
 </segment>
 <segment>
@@
 </segment>
 <segment>
-<pinref part="SG1" gate="G$1" pin="2"/>
 <pinref part="GND10" gate="1" pin="GND"/>
 <wire x1="104.14" y1="25.4" x2="104.14" y2="22.86" width="0.1524" layer="91"/>
+<pinref part="SG1" gate="G$1" pin="2"/>
 </segment>
 </net>
@@
 <wire x1="-5.08" y1="63.5" x2="-10.16" y2="63.5" width="0.1524" layer="91"/>
 <pinref part="TR1" gate="G$1" pin="1"/>
-<pinref part="S2" gate="BEF1" pin="O"/>
 <wire x1="-10.16" y1="63.5" x2="-13.97" y2="63.5" width="0.1524" layer="91"/>
 <wire x1="-22.86" y1="73.66" x2="-10.16" y2="73.66" width="0.1524" layer="91"/>
 <wire x1="-10.16" y1="73.66" x2="-10.16" y2="63.5" width="0.1524" layer="91"/>
 <junction x="-10.16" y="63.5"/>
+<pinref part="S3" gate="1" pin="O"/>
 </segment>
 </net>
@@
 <net name="N$17" class="0">
 <segment>
-<pinref part="S3" gate="G$1" pin="2"/>
 <pinref part="TR3" gate="G$1" pin="2"/>
 <wire x1="134.62" y1="30.48" x2="134.62" y2="27.94" width="0.1524" layer="91"/>
 <wire x1="134.62" y1="27.94" x2="135.89" y2="27.94" width="0.1524" layer="91"/>
+<pinref part="S1" gate="1" pin="P@1"/>
 </segment>
 </net>
@@
 <wire x1="121.92" y1="15.24" x2="121.92" y2="45.72" width="0.1524" layer="91"/>
 <wire x1="121.92" y1="45.72" x2="134.62" y2="45.72" width="0.1524" layer="91"/>
-<pinref part="S3" gate="G$1" pin="4"/>
 <wire x1="134.62" y1="45.72" x2="134.62" y2="40.64" width="0.1524" layer="91"/>
+<pinref part="S1" gate="1" pin="S@1"/>
 </segment>
 </net>
@@
 <segment>
 <pinref part="IC1" gate="G$1" pin="(PCI23/AIN1)PD7"/>
-<pinref part="SG1" gate="G$1" pin="1"/>
 <wire x1="50.8" y1="20.32" x2="96.52" y2="20.32" width="0.1524" layer="91"/>
 <wire x1="96.52" y1="20.32" x2="96.52" y2="25.4" width="0.1524" layer="91"/>
+<pinref part="SG1" gate="G$1" pin="1"/>
 </segment>
 </net>
@@
 packages will not be understood (or retained) with this version.
 </note>
+<note version="9.4" severity="warning">
+Since Version 9.4, EAGLE supports the overriding of 3D packages
+in schematics and board files. Those overridden 3d packages
+will not be understood (or retained) with this version.
+</note>
 </compatibility>
